File: Circuits/LRE_Xiao_Addon/LRE_Xiao_Addon.kicad_pcb (KiCad board)
At the start: 2 copper layers, 25 x 25 mm, 14 parts, among them J1 Conn_01x06_Socket, J3 Conn_01x06_Socket, J4 Conn_01x02_Pin, Q1 S8050, Q2 S8050, Q3 S8050

Commit message: PCB v0.5
Parts:
- added J2: Conn_01x02_Socket, Connector_PinHeader_2.54mm:PinHeader_1x02_P2.54mm_Vertical, F.Cu at (25.2, 15.3)
- added R7: 200k, Resistor_SMD:R_0805_2012Metric_Pad1.20x1.40mm_HandSolder, F.Cu at (23.6, 34.0)
- added R8: 200k, Resistor_SMD:R_0805_2012Metric_Pad1.20x1.40mm_HandSolder, F.Cu at (23.6, 32.0)
- R4, R6: value 5 -> 11
- R5: value 40 -> 61
- moved R6 3.61 mm to (30.0, 28.9)
- moved R3 3.52 mm to (20.1, 29.1)
- moved Q3 2.66 mm to (27.1, 33.0)
- moved R4 1.00 mm to (29.9, 24.0)
- moved Q2 0.92 mm to (29.3, 17.1)
- moved R2 0.90 mm to (28.4, 19.9)
- moved R5 0.88 mm to (20.9, 24.1)
- moved Q1 0.85 mm to (21.2, 17.1)
Connections:
- J1 pad 1: Net-(J1-Pin_1) -> unconnected-(J1-Pin_1-Pad1)
- J1 pad 3: Net-(J1-Pin_3) -> unconnected-(J1-Pin_3-Pad3)
- J1 pad 5: unconnected-(J1-Pin_5-Pad5) -> Net-(J1-Pin_5)
- J1 pad 6: unconnected-(J1-Pin_6-Pad6) -> Net-(J1-Pin_6)
- J3 pad 4: unconnected-(J3-Pin_4-Pad4) -> Net-(J3-Pin_4)
- J4 pad 1: Net-(J1-Pin_4) -> Net-(J3-Pin_4)
- R1 pad 1: Net-(J1-Pin_1) -> Net-(J1-Pin_4)
- R2 pad 1: Net-(J1-Pin_2) -> Net-(J1-Pin_5)
- R3 pad 1: Net-(J1-Pin_3) -> Net-(J1-Pin_6)
Routing:
- net Net-(J2-Pin_2): track 0.00 -> 40.0 mm, vias 0 -> 1
- net Net-(J2-Pin_1): track 0.00 -> 36.1 mm, vias 0 -> 1
- net Net-(J1-Pin_5): track 0.00 -> 17.7 mm
- net Net-(Q3-B): track 4.39 -> 21.5 mm
- net Net-(J1-Pin_3): track 13.9 -> 0.00 mm
- net Net-(J3-Pin_4): track 0.00 -> 8.62 mm
- net Net-(J1-Pin_2): track 9.08 -> 15.1 mm
- net Net-(D5-AR): track 8.07 -> 2.81 mm
- net Net-(Q2-B): track 9.73 -> 4.83 mm
- net Net-(D5-AB): track 4.25 -> 0.30 mm, vias 1 -> 0
- net Net-(J1-Pin_1): track 3.63 -> 0.00 mm
- net Net-(J1-Pin_6): track 0.00 -> 2.89 mm
- net Net-(D5-KG): track 6.85 -> 9.42 mm
- net VCC: track 23.1 -> 20.5 mm
- net GND: track 48.2 -> 46.3 mm, vias 2 -> 1
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Other:
- board text added: "V0.5"
- board text removed: "V0.4"

Commit message: smol fixes
Routing:
- net Net-(D5-AR): track 2.81 -> 8.17 mm
- net Net-(D5-AB): track 0.30 -> 4.48 mm, vias 0 -> 1
- net VCC: track 20.5 -> 18.8 mm
Changed lines of the file:
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@@
+	)
+	(segment
+		(start 27.5 21.75)
+		(end 28.5 21.75)
+		(width 0.25)
+		(layer "F.Cu")
+		(net 3)
+	)
+	(segment
+		(start 27.2 22.05)
+		(end 27.5 21.75)
+		(width 0.25)
+		(layer "F.Cu")
+		(net 3)
+	)
+	(segment
+		(start 27.2 23.12)
+		(end 27.2 22.05)
+		(width 0.25)
+		(layer "F.Cu")
+		(net 3)
+	)
+	(via
+		(at 28.5 21.75)
+		(size 0.8)
+		(drill 0.4)
+		(layers "F.Cu" "B.Cu")
+		(net 3)
+	)
+	(segment
+		(start 29.2 21.75)
+		(end 29.9 22.45)
+		(width 0.25)
+		(layer "B.Cu")
+		(net 3)
+	)
+	(segment
+		(start 28.5 21.75)
+		(end 29.2 21.75)
+		(width 0.25)
+		(layer "B.Cu")
+		(net 3)
 	)
 	(segment
@@
 	)
 	(segment
+		(start 24.42 24.92)
+		(end 25 24.92)
+		(width 0.25)
+		(layer "B.Cu")
+		(net 6)
+	)
+	(segment
+		(start 23.5 24)
+		(end 24.42 24.92)
+		(width 0.25)
+		(layer "B.Cu")
+		(net 6)
+	)
+	(segment
+		(start 22 24)
+		(end 23.5 24)
+		(width 0.25)
+		(layer "B.Cu")
+		(net 6)
+	)
+	(segment
+		(start 20.85 22.85)
+		(end 22 24)
+		(width 0.25)
+		(layer "B.Cu")
+		(net 6)
+	)
+	(segment
+		(start 20.85 22.5)
+		(end 20.85 22.85)
+		(width 0.25)
+		(layer "B.Cu")
+		(net 6)
+	)
+	(segment
 		(start 22.1875 16.1)
 		(end 23.55 17.4625)
@@
 	)
 	(segment
-		(start 31.824 24.676)
-		(end 33 23.5)
-		(width 0.25)
-		(layer "F.Cu")
-		(net 19)
-	)
-	(segment

Commit message: v0.51
Routing:
- net GND: track 46.3 -> 47.7 mm
Changed lines of the file:
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@@
-	)
-	(segment
-		(start 26.2 31.1)
-		(end 27.15 32.05)
-		(width 0.25)
-		(layer "F.Cu")
-		(net 2)
-	)
-	(segment
-		(start 22.059 29.809)
-		(end 23.35 31.1)
-		(width 0.25)
-		(layer "F.Cu")
-		(net 2)
 	)
 	(segment
@@
 	)
 	(segment
-		(start 23.35 31.1)
-		(end 26.2 31.1)
+		(start 23 30.75)
+		(end 25.85 30.75)
+		(width 0.25)
+		(layer "F.Cu")
+		(net 2)
+	)
+	(segment
+		(start 22.059 29.809)
+		(end 23 30.75)
+		(width 0.25)
+		(layer "F.Cu")
+		(net 2)
+	)
+	(segment
+		(start 25.85 30.75)
+		(end 27.15 32.05)
 		(width 0.25)
 		(layer "F.Cu")
@@
 	)
 	(segment
+		(start 31.5 28)
+		(end 31.124 28.376)
+		(width 0.25)
+		(layer "F.Cu")
+		(net 8)
+	)
+	(segment
+		(start 33 20.96)
+		(end 31.5 22.46)
+		(width 0.25)
+		(layer "F.Cu")
+		(net 8)
+	)
+	(segment
+		(start 31.5 22.46)
+		(end 31.5 28)
+		(width 0.25)
+		(layer "F.Cu")
+		(net 8)
+	)
+	(segment
 		(start 32.06 20.96)
 		(end 33 20.96)
@@
 	)
 	(segment
-		(start 31.15 31.6)
+		(start 23.25 29.25)
+		(end 23.235 29.25)
+		(width 0.25)
+		(layer "F.Cu")
+		(net 8)
+	)
+	(segment
+		(start 31.5 31.25)
 		(end 30.5 32.25)
-		(width 0.25)
-		(layer "F.Cu")
-		(net 8)
-	)
-	(segment
-		(start 29.775 32.25)
-		(end 28.764822 32.25)
-		(width 0.25)
-		(layer "F.Cu")
-		(net 8)
-	)
-	(segment
-		(start 33 20.96)
-		(end 31.15 22.81)
-		(width 0.25)
-		(layer "F.Cu")
-		(net 8)
-	)
-	(segment
-		(start 28.764822 32.25)
-		(end 26.940822 30.426)
 		(width 0.25)
 		(layer "F.Cu")
@@
 	)
 	(segment
-		(start 26.940822 30.426)
-		(end 24.411 30.426)
+		(start 25.407976 21.669)
+		(end 26.626976 20.45)
+		(width 0.25)
+		(layer "F.Cu")
+		(net 8)
+	)
+	(segment
+		(start 28.60072 27.874)
+		(end 24.611 27.874)
+		(width 0.25)
+		(layer "F.Cu")
+		(net 8)
+	)
+	(segment
+		(start 24.611 27.874)
+		(end 23.235 29.25)
+		(width 0.25)
+		(layer "F.Cu")
+		(net 8)
+	)
+	(segment
+		(start 29.10272 28.376)
+		(end 28.60072 27.874)
+		(width 0.25)
+		(layer "F.Cu")
+		(net 8)
+	)
+	(segment
+		(start 31.55 20.45)
+		(end 32.06 20.96)
+		(width 0.25)
+		(layer "F.Cu")
+		(net 8)
+	)
+	(segment
+		(start 26.626976 20.45)
+		(end 31.55 20.45)
+		(width 0.25)
+		(layer "F.Cu")
+		(net 8)
+	)
+	(segment
+		(start 31.5 28)
+		(end 31.5 31.25)
 		(width 0.25)
 		(layer "F.Cu")
@@
 	)
 	(segment
-		(start 25.407976 21.669)
-		(end 26.626976 20.45)
-		(width 0.25)
-		(layer "F.Cu")
-		(net 8)
-	)
-	(segment
-		(start 31.15 22.81)
-		(end 31.15 31.6)
-		(width 0.25)
-		(layer "F.Cu")
-		(net 8)
-	)
-	(segment
-		(start 24.411 30.426)
-		(end 23.235 29.25)
-		(width 0.25)
-		(layer "F.Cu")
-		(net 8)
-	)
-	(segment
-		(start 31.55 20.45)
-		(end 32.06 20.96)
-		(width 0.25)
-		(layer "F.Cu")
-		(net 8)
-	)
-	(segment
-		(start 26.626976 20.45)
-		(end 31.55 20.45)
-		(width 0.25)
-		(layer "F.Cu")
+		(start 31.124 28.376)
+		(end 29.10272 28.376)
+		(width 0.25)
+		(layer "F.Cu")
